Commit message: fully working navigation

File: src/rosbot_simulation/urdf/puck.xacro (robot description, xacro)
@@ -8,4 +8,9 @@
   <xacro:arg name="g" default="0.0"/>
   <xacro:arg name="b" default="0.0"/>
+  <!-- Gazebo material script name. Must be one of the predefined Gazebo
+       materials (e.g. Gazebo/Red, Gazebo/Green, Gazebo/Blue). The previous
+       version hardcoded Gazebo/Red here, which made every puck render red
+       and broke HSV-based colour classification in perception_node. -->
+  <xacro:arg name="gazebo_material" default="Gazebo/Red"/>
   <link name="$(arg name)_link">
     <inertial>
@@ -36,5 +41,5 @@
   </link>
   <gazebo reference="$(arg name)_link">
-    <material>Gazebo/Red</material>
+    <material>$(arg gazebo_material)</material>
   </gazebo>
 </robot>
